Commit message: revised from lexus to aidi_axio

File: urdf/vehicle.xacro (robot description, xacro)
@@ -2,5 +2,5 @@
 <robot xmlns:xacro="http://ros.org/wiki/xacro">
   <!-- load parameter -->
-  <xacro:property name="vehicle_info" value="${load_yaml('$(find lexus_description)/config/vehicle_info.yaml')}"/>
+  <xacro:property name="vehicle_info" value="${load_yaml('$(find aidi_axio_description)/config/vehicle_info.yaml')}"/>
   <!-- vehicle body -->
   <link name="base_link">

Commit message: revised from lexus to aidi_axio

File: urdf/vehicle.xacro (robot description, xacro)
@@ -8,5 +8,5 @@
       <origin xyz="${vehicle_info['wheel_base']/2.0} 0 0" rpy="${pi/2.0} 0 ${pi}"/>
       <geometry>
-        <mesh filename="package://lexus_description/mesh/lexus.dae" scale="1 1 1"/>
+        <mesh filename="package://aidi_axio_description/mesh/lexus.dae" scale="1 1 1"/>
       </geometry>
     </visual>
